File: hardware/kicad/4key/4key.kicad_sch (KiCad schematic)
At the start: 35 parts, among them J1 USB_C_Receptacle, J2 SPARE / DEBUG, SW1 AGENT1, SW2 AGENT2, SW3 AGENT3, SW4 PTT, U1 ESP32-S3-WROOM-1-N16R8, U2 XL9555 / PCF8575 (TSSOP-24), U3 AP2112K-3.3, U4 74LVC1G17

Commit message: Fix real generator bugs found by an independent pre-fab hardware review
Verified all 41 ESP32-S3-WROOM-1 pins and all 24 XL9555 pins in
boarddef.py against their primary-source datasheets (not search-engine
summaries, which were caught being wrong twice: once claiming XL9555's
SDA/SCL were swapped, once claiming two WROOM-1 GND/thermal pins were
GPIOs). Both parts' full pin assignments match exactly.

An independent Opus review of the whole design caught three real issues
a pinout check alone couldn't:

- gen_pcb.py ignored a part's `nc` (no-connect) list entirely, while
  gen_sch.py respected it - real schematic/PCB drift for any pin that
  has both a plausible net name and an explicit no-connect (the last
  LED's DOUT, still called LEDCH%d with nothing next in the chain).
  Fixed by checking nc first in place_parts(), same as gen_sch.py.
- No bulk cap at U1's own +3V3 pin (nearest was ~37mm away). Added C9
  (10uF), T-tapped off the existing +3V3 B.Cu trunk - not literally at
  the pin, since the whole left margin is already packed solid; see the
  code comments for exactly where it landed and why.
- No USB ESD protection. Added D_ESD (USBLC6-2SC6 TVS array), pinout
  confirmed against the actual symbol KiCad ships, shunted across the
  existing USB_DP/USB_DM/+5V/GND nets. Left unrouted like the rest of
  the differential pair - this only adds the part to the schematic/BOM.

Also fixed a doc bug (gen_pcb.py's own comment on the mounting-hole
x-position didn't match the code) and a missing sym-lib-table entry for
the new ESD diode's symbol library.

All three tiers (4key/8key/12key) regenerated and re-verified: 0 DRC
violations, 0 ERC violations.

One real gap surfaced, not a code fix: boarddef.py's LED footprint
(plain SK6812MINI, not "-E") is internally consistent, but the
current-budget math elsewhere was computed against the wrong datasheet
("-E"'s) - needs the exact SKU locked down before ordering. Also
confirmed no enclosure/case file exists in this repo at a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
Parts:
- added C9: 10u, Capacitor_SMD:C_0805_2012Metric_Pad1.18x1.45mm_HandSolder, symbol Device:C
- added D_ESD: USBLC6-2SC6, Package_TO_SOT_SMD:SOT-23-6, symbol Power_Protection:USBLC6-2SC6
Connections:
- net +3V3: now also C9.1
- net +5V: now also D_ESD.5 (VBUS)
- net GND: now also C9.2, D_ESD.2 (GND)
- net USB_DM: now also D_ESD.1 (I/O1), D_ESD.6 (I/O1)
- net USB_DP: now also D_ESD.3 (I/O2), D_ESD.4 (I/O2)
