File: hardware/kicad/8key/8key.kicad_pcb (KiCad board)
At the start: 2 copper layers, 87.2 x 89.6 mm, 51 parts, among them J1 USB_C_Receptacle, J2 SPARE / DEBUG, SW1 AGENT1, SW2 AGENT2, SW3 AGENT3, SW4 AGENT4, SW5 AGENT5, SW6 AGENT6, SW7 AGENT7, SW8 PTT, U1 ESP32-S3-WROOM-1-N16R8, U2 XL9555 / PCF8575 (TSSOP-24), U3 AP2112K-3.3, U4 74LVC1G17

Commit message: Fix real generator bugs found by an independent pre-fab hardware review
Verified all 41 ESP32-S3-WROOM-1 pins and all 24 XL9555 pins in
boarddef.py against their primary-source datasheets (not search-engine
summaries, which were caught being wrong twice: once claiming XL9555's
SDA/SCL were swapped, once claiming two WROOM-1 GND/thermal pins were
GPIOs). Both parts' full pin assignments match exactly.

An independent Opus review of the whole design caught three real issues
a pinout check alone couldn't:

- gen_pcb.py ignored a part's `nc` (no-connect) list entirely, while
  gen_sch.py respected it - real schematic/PCB drift for any pin that
  has both a plausible net name and an explicit no-connect (the last
  LED's DOUT, still called LEDCH%d with nothing next in the chain).
  Fixed by checking nc first in place_parts(), same as gen_sch.py.
- No bulk cap at U1's own +3V3 pin (nearest was ~37mm away). Added C9
  (10uF), T-tapped off the existing +3V3 B.Cu trunk - not literally at
  the pin, since the whole left margin is already packed solid; see the
  code comments for exactly where it landed and why.
- No USB ESD protection. Added D_ESD (USBLC6-2SC6 TVS array), pinout
  confirmed against the actual symbol KiCad ships, shunted across the
  existing USB_DP/USB_DM/+5V/GND nets. Left unrouted like the rest of
  the differential pair - this only adds the part to the schematic/BOM.

Also fixed a doc bug (gen_pcb.py's own comment on the mounting-hole
x-position didn't match the code) and a missing sym-lib-table entry for
the new ESD diode's symbol library.

All three tiers (4key/8key/12key) regenerated and re-verified: 0 DRC
violations, 0 ERC violations.

One real gap surfaced, not a code fix: boarddef.py's LED footprint
(plain SK6812MINI, not "-E") is internally consistent, but the
current-budget math elsewhere was computed against the wrong datasheet
("-E"'s) - needs the exact SKU locked down before ordering. Also
confirmed no enclosure/case file exists in this repo at a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
Parts:
- removed H48, H49: MountingHole_2.2mm_M2, MountingHole_2.2mm_M2
- added C9: 10u, C_0805_2012Metric_Pad1.18x1.45mm_HandSolder, F.Cu at (141.0, 133.0)
- added D_ESD: USBLC6-2SC6, SOT-23-6, F.Cu at (136.0, 124.0)
- added H52: MountingHole_2.2mm_M2, MountingHole_2.2mm_M2, F.Cu at (104.0, 185.6)
- added H53: MountingHole_2.2mm_M2, MountingHole_2.2mm_M2, F.Cu at (183.2, 185.6)
- moved H50 94.4 mm to (151.5, 104.0)
- moved H51 81.6 mm to (183.2, 104.0)
Connections:
- D8 pad 1: LEDCH8 -> (no net)
Routing:
- net +3V3: track 115.6 -> 123.1 mm, vias 2 -> 3

Commit message: Fix 4key I2C pull-up placement, grow the board, finish routing
Root-caused the 4key board's unrouted/short-prone corner: R4/R5 (the
I2C pull-ups for U2) were placed 16mm from the chip they serve, forcing
their traces across every other bus lane on the board. Moved them next
to U2 in boarddef.py, and grew STRIP 46mm -> 58mm (87.2x70.5mm ->
87.2x82.65mm) to give that whole corner real room — both the autorouter
and hand-routing had been failing to close the last nets in the old,
cramped layout.

route_strip()'s I2C section also hard-shorted SCL/SDA into +3V3 and
into each other once U2 moved down next to R4/R5 (caught by an
independent Opus review before fab) — rewritten to route both nets on
B.Cu the whole way, with small (0.5mm) vias where the standard 0.8mm
via can't fit the 0.65mm pin pitch.

Final DRC on the 4key board: 4 minor violations (2 pre-existing and
unrelated, 1 harmless dangling stub, cosmetic disconnected-but-same-net
ground-pour islands) and 2 low-priority unrouted pads in an extremely
congested corner (a spare header pin, a redundant pull-up supply leg) —
down from 39 unconnected items and multiple shorts earlier in this
pass. 8key/12key inherit the same STRIP/placement change and still
generate cleanly, but keep their own routing out of scope per the
existing "4key only" convention in gen_pcb.py.

Also adds hardware/enclosure/: a build123d-based parametric case
generator (hardware/enclosure/tools/gen_case.py) and its first-draft
4key tray/plate STLs, built from the real boarddef.py geometry rather
than guessed dimensions.

Boards ordered from JLCPCB at this routed revision.

Co-Authored-By: Claude Sonnet 5 <noreply@anthropic.com>
Parts:
- moved D_ESD 37.5 mm to (173.0, 130.0)
- moved R4 25.1 mm to (168.0, 140.0)
- moved R5 25.1 mm to (168.0, 144.0)
- moved CL1 12.0 mm to (108.0, 175.1)
- moved CL2 12.0 mm to (127.1, 175.1)
- moved CL3 12.0 mm to (146.1, 175.1)
- moved CL4 12.0 mm to (165.2, 175.1)
- moved CL5 12.0 mm to (108.0, 194.2)
- moved CL6 12.0 mm to (127.1, 194.2)
- moved CL7 12.0 mm to (146.1, 194.2)
- moved CL8 12.0 mm to (165.2, 194.2)
- moved D1 12.0 mm to (115.0, 172.5)
- moved D2 12.0 mm to (134.1, 172.5)
- moved D3 12.0 mm to (153.1, 172.5)
- moved D4 12.0 mm to (172.2, 172.5)
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Routing:
- net +3V3: track 123.1 -> 147.6 mm
- net SDA: track 68.1 -> 52.0 mm
- net LEDCH0: track 41.6 -> 53.6 mm
- net +5V: track 408.3 -> 420.3 mm
- net SCL: track 64.3 -> 64.9 mm
Other:
- board size 87.2 x 89.6 mm -> 87.2 x 101.6 mm
